Commit message: turn test/SharedMemory/test.c into a gtest for CI unit testing in github remove overly verbose printfs in importers fix axis in r2d2.urdf

File: data/r2d2.urdf (robot description, URDF)
Before this commit: robot physics, 16 links, 15 joints
Joints:
- joint gripper_extension: axis (none) -> 0 0 1

Commit message: fix axis in r2d2.urdf enable SimpleOpenGL3 demo for CMake

File: data/r2d2.urdf (robot description, URDF)
Before this commit: robot physics, 16 links, 15 joints
Joints:
- joint gripper_extension: axis 0 0 1 -> 1 0 0
