Commit message: Physics runs in a separate thread from rendering in PhysicsServerExample (preliminary) Improve rendering performance. OpenVR experience is smooth now. commit needs a bit more testing before pushing in main repo.

File: data/sphere2.urdf (robot description, URDF)
Before this commit: robot urdf_robot, 3 links, 2 joints
Links:
- removed link childA
- removed link childB
Joints:
- removed joint joint_baseLink_childA
- removed joint joint_childA_childB
