Commit message: prepare robotics learning examples, see examples/RoboticsLearning/b3RobotSimAPI.h prepare compliant contact work, urdf loading of parameters (see data/cube.urdf)

File: data/cube.urdf (robot description, URDF)
Before this commit: robot urdf_robot, 1 links, 0 joints
Links:
- link baseLink: mass 10.0 -> 1.0; geometry collision box size=1 1 1; visual mesh filename=cube.obj scale=1 1 1
