Commit message: Add rolling friction, set rolling friction coefficient from urdf, and set up two point contact experiment.

File: data/cube_gripper_left.urdf (robot description, URDF)
Before this commit: robot cube.urdf, 1 links, 0 joints
Links:
- added link world
Joints:
- added joint cube_joint: type prismatic, parent world, child baseLink, origin xyz=0 0 0 rpy=0 0 0, axis 1 0 0, limit lower=-2.96705972839 upper=2.96705972839 effort=300 velocity=10

File: data/cube_gripper_right.urdf (robot description, URDF)
Before this commit: robot cube.urdf, 1 links, 0 joints
Links:
- added link world
Joints:
- added joint cube_joint: type prismatic, parent world, child baseLink, origin xyz=0 0 0 rpy=0 0 0, axis 1 0 0, limit lower=-2.96705972839 upper=2.96705972839 effort=300 velocity=10
