Commit message: remove that odd triangle in the origin of samurai castle (VR) add rolling/spinning friction to cube, remove it from plane/samurai.urdf URDF2Bullet: support joint limits for revolute and prismatic, only if defined (if upper < lower, disable limit) add some profiling markers to improve performance

File: data/plane.urdf (robot description, URDF)
Before this commit: robot cube.urdf, 1 links, 0 joints
Links:
- removed link baseLink
- added link planeLink, mass .0; collision box size=10 10 0.001; visual mesh filename=plane.obj scale=1 1 1

File: data/pr2_gripper.urdf (robot description, URDF)
Before this commit: robot physics, 5 links, 4 joints
Links:
- link gripper_pole: mass 0.05 -> 100
- link left_gripper: geometry visual mesh filename=l_finger.stl
- link left_tip: geometry collision box size=.13 .03 .02; visual mesh filename=l_finger_tip.stl
- link right_gripper: geometry visual mesh filename=l_finger.stl
- link right_tip: geometry collision box size=.13 .03 .02; visual mesh filename=l_finger_tip.stl

File: data/teddy_vhacd.urdf (robot description, URDF)
Before this commit: robot cube.urdf, 1 links, 0 joints
Links:
- link baseLink: mass .1 -> 1.0; geometry collision mesh filename=teddy2_VHACD_CHs.obj scale=1 1 1; visual mesh filename=teddy2_VHACD_CHs.obj scale=1 1 1
