Commit message: Add small sphere, make teddy small too Add physics time scale in VR mode Fix compound collision margin in physics server Enable visuals for rigid body (non-multi-body) URDF/SDF loading in physics server.

File: data/teddy_vhacd.urdf (robot description, URDF)
Before this commit: robot cube.urdf, 1 links, 0 joints
Links:
- link baseLink: mass 1.0 -> .1; geometry collision mesh filename=teddy2_VHACD_CHs.obj scale=.1 .1 .1; visual mesh filename=teddy2_VHACD_CHs.obj scale=.1 .1 .1
