Commit message: rolling friction -> combine using rolling*normal friction, add for both objects. rolling friction -> only along the normal, until we have separate rolling friction coefficients on normal and non-normal directions Don't teleport with grasping controller (VR) Tune VR grasping a bit.

File: data/pr2_gripper.urdf (robot description, URDF)
Before this commit: robot physics, 5 links, 4 joints
Links:
- link left_tip: geometry collision box size=.03 .03 .02; visual mesh filename=l_finger_tip.stl
- link right_tip: geometry collision box size=.03 .03 .02; visual mesh filename=l_finger_tip.stl

Commit message: tune gripper parameters for VR demo

File: data/pr2_gripper.urdf (robot description, URDF)
Before this commit: robot physics, 5 links, 4 joints
Links:
- link gripper_pole: mass 100 -> 0.5
- link left_gripper: mass 0.05 -> 0.5; geometry collision mesh filename=l_finger_collision.stl scale=.9 .9 .9; visual mesh filename=l_finger.stl
- link left_tip: mass 0.05 -> 0.1; geometry collision box size=.03 .03 .02; visual mesh filename=l_finger_tip.stl
- link right_gripper: geometry collision mesh filename=l_finger_collision.stl scale=.9 .9 .9; visual mesh filename=l_finger.stl
- link right_tip: geometry collision box size=.03 .03 .02; visual mesh filename=l_finger_tip.stl

Commit message: more tweak in pr2_gripper.urdf (VR), remove some collision meshes (until interaction issues are resolved)

File: data/pr2_gripper.urdf (robot description, URDF)
Before this commit: robot physics, 5 links, 4 joints
Links:
- link left_gripper: geometry visual mesh filename=l_finger.stl
- link left_tip: mass 0.1 -> 0.05
- link right_gripper: geometry visual mesh filename=l_finger.stl

Commit message: decrease some gjk/epa tolerance to improve collision detection using very small collision margins (0.001/1mm) tweak pr2 gripper.

File: data/pr2_gripper.urdf (robot description, URDF)
Before this commit: robot physics, 5 links, 4 joints
Links:
- link left_gripper: mass 0.5 -> 0.1; geometry collision mesh filename=l_finger_collision.stl; visual mesh filename=l_finger_collision.stl
- link left_tip: mass 0.05 -> 0.1
- link right_gripper: mass 0.05 -> 0.1; geometry collision mesh filename=l_finger_collision.stl; visual mesh filename=l_finger_collision.stl
- link right_tip: mass 0.05 -> 0.1

Commit message: better pr2_gripper collision model

File: data/pr2_gripper.urdf (robot description, URDF)
Before this commit: robot physics, 5 links, 4 joints
Links:
- link left_tip: geometry collision box size=.03 .01 .02; visual mesh filename=l_finger_tip.stl
- link right_tip: geometry collision box size=.01 .02 .02; collision box size=.03 .01 .02
