Commit message: Implement first draft of pybullet.createVisualShape and add createVisualShape.py example add normals to duck.obj for nicer appearance fix plane100.urdf (so collision shape matches visual shape size)

File: data/plane100.urdf (robot description, URDF)
Before this commit: robot cube.urdf, 1 links, 0 joints
Links:
- link baseLink: geometry collision box size=200 200 0.001; visual mesh filename=plane100.obj scale=1 1 1
