Commit message: add test end-effector for Kuka iiwa (IK)

File: data/kuka_iiwa/model.urdf (robot description, URDF)
Before this commit: robot lbr_iiwa, 8 links, 7 joints
Links:
- added link lbr_iiwa_link_endeffector, mass 0.3
Joints:
- added joint lbr_iiwa_joint_8: type fixed, parent lbr_iiwa_link_7, child lbr_iiwa_link_endeffector, origin xyz=0 0.0 0.08 rpy=0 0 0, axis 0 0 1

Commit message: URDF: don't parse joint limit for continuous joints tweak KUKA iiwa inverse kinematics test in physics server

File: data/kuka_iiwa/model.urdf (robot description, URDF)
Before this commit: robot lbr_iiwa, 9 links, 8 joints
Links:
- removed link lbr_iiwa_link_endeffector
Joints:
- removed joint lbr_iiwa_joint_8

Commit message: expose b3PhysicsParamSetNumSolverIterations split Visual Studio project generation batch file in regular and VR+pybullet+double precision build. disable KUKA iiwa joint limit hack

File: data/kuka_iiwa/model.urdf (robot description, URDF)
Before this commit: robot lbr_iiwa, 8 links, 7 joints
Joints:
- joint lbr_iiwa_joint_4: limit lower=.29439510239 upper=2.09439510239 effort=300 velocity=10 -> lower=-2.09439510239 upper=2.09439510239 effort=300 velocity=10
