Commit message: update minitaur.py to use minitaur.urdf (instead of quadruped.urdf), also sort the legs in the same order as real hardware added test urdf files for minitaur with all fixed joints, or fixed knees. added some stiffness/damping to minitaur legs (testing) tiny_obj_loader, don't crash on invalid texture coordinates btMultiBodyConstraintSolver: sweep back and forward to reduce asymmetry

File: data/quadruped/minitaur_fixed_all.urdf (robot description, URDF)
Before this commit: robot quadruped, 27 links, 26 joints
Joints:
- joint knee_back_leftL_link: origin xyz=0.0 0.01 .055 rpy=0 0 0 -> xyz=0.0 0.01 .055 rpy=0 2.1834 0; type revolute -> fixed
- joint knee_back_leftR_link: origin xyz=0.0 0.01 .055 rpy=0 0 0 -> xyz=0.0 0.01 .055 rpy=0 2.1834 0; type revolute -> fixed
- joint knee_back_rightL_link: origin xyz=0.0 0.01 .055 rpy=0 0 0 -> xyz=0.0 0.01 .055 rpy=0 -2.1834 0; type revolute -> fixed
- joint knee_back_rightR_link: origin xyz=0.0 0.01 .055 rpy=0 0 0 -> xyz=0.0 0.01 .055 rpy=0 -2.1834 0; type revolute -> fixed
- joint knee_front_leftL_link: origin xyz=0.0 0.01 .055 rpy=0 0 0 -> xyz=0.0 0.01 .055 rpy=0 2.1834 0; type revolute -> fixed
- joint knee_front_leftR_link: origin xyz=0.0 0.01 .055 rpy=0 0 0 -> xyz=0.0 0.01 .055 rpy=0 2.1834 0; type revolute -> fixed
- joint knee_front_rightL_link: origin xyz=0.0 0.01 .055 rpy=0 0 0 -> xyz=0.0 0.01 .055 rpy=0 -2.1834 0; type revolute -> fixed
- joint knee_front_rightR_link: origin xyz=0.0 0.01 .055 rpy=0 0 0 -> xyz=0.0 0.01 .055 rpy=0 -2.1834 0; type revolute -> fixed
- joint motor_back_leftL_joint: origin xyz=-0.21 -0.04 0 rpy=1.57075 0 0 -> xyz=-0.21 -0.04 0 rpy=1.57075 1.570796 0; type continuous -> fixed
- joint motor_back_leftR_joint: origin xyz=-0.21 0.025 0 rpy=1.57075 0 3.141592 -> xyz=-0.21 0.025 0 rpy=1.57075 1.570796 3.141592; type continuous -> fixed
- joint motor_back_rightL_joint: origin xyz=-0.21 0.04 0 rpy=1.57075 0 3.141592 -> xyz=-0.21 0.04 0 rpy=1.57075 -1.570796 3.141592; type continuous -> fixed
- joint motor_back_rightR_joint: origin xyz=-0.21 -0.025 0 rpy=1.57075 0 0 -> xyz=-0.21 -0.025 0 rpy=1.57075 -1.570796 0; type continuous -> fixed
- joint motor_front_leftL_joint: origin xyz=0.21 -0.04 0 rpy=1.57075 0 0 -> xyz=0.21 -0.04 0 rpy=1.57075 1.570796 0; type continuous -> fixed
- joint motor_front_leftR_joint: origin xyz=0.21 0.025 0 rpy=1.57075 0 3.141592 -> xyz=0.21 0.025 0 rpy=1.57075 1.570796 3.141592; type continuous -> fixed
- joint motor_front_rightL_joint: origin xyz=0.21 0.04 0 rpy=1.57075 0 3.141592 -> xyz=0.21 0.04 0 rpy=1.57075 -1.570796 3.141592; type continuous -> fixed
- joint motor_front_rightR_joint: origin xyz=0.21 -0.025 0 rpy=1.57075 0 0 -> xyz=0.21 -0.025 0 rpy=1.57075 -1.570796 0; type continuous -> fixed

File: data/quadruped/minitaur_fixed_knees.urdf (robot description, URDF)
Before this commit: robot quadruped, 27 links, 26 joints
Joints:
- joint knee_back_leftL_link: origin xyz=0.0 0.01 .055 rpy=0 0 0 -> xyz=0.0 0.01 .055 rpy=0 2.1834 0; type revolute -> fixed
- joint knee_back_leftR_link: origin xyz=0.0 0.01 .055 rpy=0 0 0 -> xyz=0.0 0.01 .055 rpy=0 2.1834 0; type revolute -> fixed
- joint knee_back_rightL_link: origin xyz=0.0 0.01 .055 rpy=0 0 0 -> xyz=0.0 0.01 .055 rpy=0 -2.1834 0; type revolute -> fixed
- joint knee_back_rightR_link: origin xyz=0.0 0.01 .055 rpy=0 0 0 -> xyz=0.0 0.01 .055 rpy=0 -2.1834 0; type revolute -> fixed
- joint knee_front_leftL_link: origin xyz=0.0 0.01 .055 rpy=0 0 0 -> xyz=0.0 0.01 .055 rpy=0 2.1834 0; type revolute -> fixed
- joint knee_front_leftR_link: origin xyz=0.0 0.01 .055 rpy=0 0 0 -> xyz=0.0 0.01 .055 rpy=0 2.1834 0; type revolute -> fixed
- joint knee_front_rightL_link: origin xyz=0.0 0.01 .055 rpy=0 0 0 -> xyz=0.0 0.01 .055 rpy=0 -2.1834 0; type revolute -> fixed
- joint knee_front_rightR_link: origin xyz=0.0 0.01 .055 rpy=0 0 0 -> xyz=0.0 0.01 .055 rpy=0 -2.1834 0; type revolute -> fixed
