Commit message: make the URDF and the minitaur.py consistent with the real robot

File: data/quadruped/minitaur.urdf (robot description, URDF)
Before this commit: robot quadruped, 27 links, 26 joints
Links:
- link base_chassis_link: geometry collision box size=.17 0.10 .05; collision box size=.17 0.10 .05
- link motor_front_leftL_link: geometry collision cylinder length=0.026 radius=0.0434; visual mesh filename=tmotor3.obj scale=1 1 1
- link motor_front_leftR_link: geometry visual mesh filename=tmotor3.obj scale=1 1 1
Joints:
- joint motor_back_leftL_joint: origin xyz=-0.21 -0.04 0 rpy=1.57075 0 0 -> xyz=-0.21 0.025 0 rpy=1.57075 0 3.141592
- joint motor_back_leftR_joint: origin xyz=-0.21 0.025 0 rpy=1.57075 0 3.141592 -> xyz=-0.21 -0.04 0 rpy=1.57075 0 0
- joint motor_front_leftL_joint: origin xyz=0.21 -0.04 0 rpy=1.57075 0 0 -> xyz=0.21 0.025 0 rpy=1.57075 0 3.141592
- joint motor_front_leftR_joint: origin xyz=0.21 0.025 0 rpy=1.57075 0 3.141592 -> xyz=0.21 -0.04 0 rpy=1.57075 0 0

Commit message: fix minitaur.urdf: move lower-leg inertia to center, add missing collision for one of the motors, add contact parameters for friction_anchor, spinning friction, compliance (stiffness/damping) fix in indexing for maximal coordinates (unused by default, still experimental, requires many iterations for Minitaur due to extreme mass-ratio, hence use of reduces/generalized coordinates) modify quadruped.py to test maximal coordinates wrap angular servo (positional) target within [-PI,PI] in btGeneric6DofSpring2Constraint add 'j' key to show body frames in wireframe/debug mode

File: data/quadruped/minitaur.urdf (robot description, URDF)
Before this commit: robot quadruped, 27 links, 26 joints
Links:
- link motor_front_leftR_link: geometry collision cylinder length=0.026 radius=0.0434; visual mesh filename=tmotor3.obj scale=1 1 1
Joints:
- joint knee_back_leftL_link: type revolute -> continuous
- joint knee_back_leftR_link: type revolute -> continuous
- joint knee_back_rightL_link: type revolute -> continuous
- joint knee_back_rightR_link: type revolute -> continuous
- joint knee_front_leftL_link: type revolute -> continuous
- joint knee_front_leftR_link: type revolute -> continuous
- joint knee_front_rightL_link: type revolute -> continuous
- joint knee_front_rightR_link: type revolute -> continuous
