Commit message: add tingnan's new minitaur urdf for derpy.

File: data/quadruped/minitaur_derpy.urdf (robot description, URDF)
Before this commit: robot quadruped, 27 links, 26 joints
Joints:
- removed joint hip_front_leftR_link
- removed joint hip_front_rightR_link
- removed joint hip_leftR_link
- removed joint hip_rightR_link
- removed joint knee_back_leftL_link
- removed joint knee_back_leftR_link
- removed joint knee_back_rightL_link
- removed joint knee_back_rightR_link
- removed joint knee_front_leftL_link
- removed joint knee_front_leftR_link
- removed joint knee_front_rightL_link
- removed joint knee_front_rightR_link
- removed joint motor_back_leftL_link
- removed joint motor_back_rightL_link
- removed joint motor_front_leftL_link
- removed joint motor_front_rightL_link
- added joint hip_back_leftL_joint: type fixed, parent motor_back_leftL_link, child upper_leg_back_leftL_link, origin xyz=0.0 0.045 -0.030 rpy=-1.57075 0 0, axis 0 0 1, limit effort=100 velocity=100
- added joint hip_back_leftR_joint: type fixed, parent motor_back_leftR_link, child upper_leg_back_leftR_link, origin xyz=0.0 0.045 -0.030 rpy=-1.57075 0 0, axis 0 0 1, limit effort=100 velocity=100
- added joint hip_back_rightL_joint: type fixed, parent motor_back_rightL_link, child upper_leg_back_rightL_link, origin xyz=0.0 0.045 -0.030 rpy=-1.57075 0 0, axis 0 0 1, limit effort=100 velocity=100
- added joint hip_back_rightR_joint: type fixed, parent motor_back_rightR_link, child upper_leg_back_rightR_link, origin xyz=0.0 0.045 -0.030 rpy=-1.57075 0 0, axis 0 0 1, limit effort=100 velocity=100
- added joint hip_front_leftL_joint: type fixed, parent motor_front_leftL_link, child upper_leg_front_leftL_link, origin xyz=0.0 0.045 -0.030 rpy=-1.57075 0 0, axis 0 0 1, limit effort=100 velocity=100
- added joint hip_front_leftR_joint: type fixed, parent motor_front_leftR_link, child upper_leg_front_leftR_link, origin xyz=0.0 0.045 -0.030 rpy=-1.57075 0 0, axis 0 0 1, limit effort=100 velocity=100
- added joint hip_front_rightL_joint: type fixed, parent motor_front_rightL_link, child upper_leg_front_rightL_link, origin xyz=0.0 0.045 -0.030 rpy=-1.57075 0 0, axis 0 0 1, limit effort=100 velocity=100
- added joint hip_front_rightR_joint: type fixed, parent motor_front_rightR_link, child upper_leg_front_rightR_link, origin xyz=0.0 0.045 -0.030 rpy=-1.57075 0 0, axis 0 0 1, limit effort=100 velocity=100
- added joint knee_back_leftL_joint: type continuous, parent upper_leg_back_leftL_link, child lower_leg_back_leftL_link, origin xyz=0.0 0.01 .056 rpy=0 0 0, axis 0 1 0, limit effort=100 velocity=100
- added joint knee_back_leftR_joint: type continuous, parent upper_leg_back_leftR_link, child lower_leg_back_leftR_link, origin xyz=0.0 0.01 .056 rpy=0 0 0, axis 0 1 0, limit effort=100 velocity=100
- added joint knee_back_rightL_joint: type continuous, parent upper_leg_back_rightL_link, child lower_leg_back_rightL_link, origin xyz=0.0 0.01 .056 rpy=0 0 0, axis 0 1 0, limit effort=100 velocity=100
- added joint knee_back_rightR_joint: type continuous, parent upper_leg_back_rightR_link, child lower_leg_back_rightR_link, origin xyz=0.0 0.01 .056 rpy=0 0 0, axis 0 1 0, limit effort=100 velocity=100
- added joint knee_front_leftL_joint: type continuous, parent upper_leg_front_leftL_link, child lower_leg_front_leftL_link, origin xyz=0.0 0.01 .056 rpy=0 0 0, axis 0 1 0, limit effort=100 velocity=100
- added joint knee_front_leftR_joint: type continuous, parent upper_leg_front_leftR_link, child lower_leg_front_leftR_link, origin xyz=0.0 0.01 .056 rpy=0 0 0, axis 0 1 0, limit effort=100 velocity=100
- added joint knee_front_rightL_joint: type continuous, parent upper_leg_front_rightL_link, child lower_leg_front_rightL_link, origin xyz=0.0 0.01 .056 rpy=0 0 0, axis 0 1 0, limit effort=100 velocity=100
- added joint knee_front_rightR_joint: type continuous, parent upper_leg_front_rightR_link, child lower_leg_front_rightR_link, origin xyz=0.0 0.01 .056 rpy=0 0 0, axis 0 1 0, limit effort=100 velocity=100

Commit message: adjust the minitaur_derpy urdf. Seperate the motor controller and the moving part of the motor.

File: data/quadruped/minitaur_derpy.urdf (robot description, URDF)
Before this commit: robot quadruped, 27 links, 26 joints
Links:
- link chassis_left: mass .72277 -> 1.3668; geometry collision box size=.068 0.0373 .060; collision box size=.068 0.0373 .060
- link chassis_right: mass .72277 -> 1.3668; geometry collision box size=.068 0.0373 .060; collision box size=.068 0.0373 .060
- link motor_back_leftL_link: mass 0.402 -> 0.241; geometry collision cylinder length=0.0165 radius=0.0425; visual mesh filename=tmotor3.obj scale=1 1 1
- link motor_back_leftR_link: mass 0.402 -> 0.241; geometry collision cylinder length=0.0165 radius=0.0425; visual mesh filename=tmotor3.obj scale=1 1 1
- link motor_back_rightL_link: mass 0.402 -> 0.241; geometry collision cylinder length=0.0165 radius=0.0425; visual mesh filename=tmotor3.obj scale=1 1 1
- link motor_back_rightR_link: mass 0.402 -> 0.241; geometry collision cylinder length=0.0165 radius=0.0425; visual mesh filename=tmotor3.obj scale=1 1 1
- link motor_front_leftL_link: mass 0.402 -> 0.241; geometry collision cylinder length=0.0165 radius=0.0425; visual mesh filename=tmotor3.obj scale=1 1 1
- link motor_front_leftR_link: mass 0.402 -> 0.241; geometry collision cylinder length=0.0165 radius=0.0425; visual mesh filename=tmotor3.obj scale=1 1 1
- link motor_front_rightL_link: mass 0.402 -> 0.241; geometry collision cylinder length=0.0165 radius=0.0425; visual mesh filename=tmotor3.obj scale=1 1 1
- link motor_front_rightR_link: mass 0.402 -> 0.241; geometry collision cylinder length=0.0165 radius=0.0425; visual mesh filename=tmotor3.obj scale=1 1 1
Joints:
- joint hip_back_leftL_joint: origin xyz=0.0 0.045 -0.030 rpy=-1.57075 0 0 -> xyz=0.0 0.045 -0.01725 rpy=-1.57075 0 0
- joint hip_back_leftR_joint: origin xyz=0.0 0.045 -0.030 rpy=-1.57075 0 0 -> xyz=0.0 0.045 -0.01725 rpy=-1.57075 0 0
- joint hip_back_rightL_joint: origin xyz=0.0 0.045 -0.030 rpy=-1.57075 0 0 -> xyz=0.0 0.045 -0.01725 rpy=-1.57075 0 0
- joint hip_back_rightR_joint: origin xyz=0.0 0.045 -0.030 rpy=-1.57075 0 0 -> xyz=0.0 0.045 -0.01725 rpy=-1.57075 0 0
- joint hip_front_leftL_joint: origin xyz=0.0 0.045 -0.030 rpy=-1.57075 0 0 -> xyz=0.0 0.045 -0.01725 rpy=-1.57075 0 0
- joint hip_front_leftR_joint: origin xyz=0.0 0.045 -0.030 rpy=-1.57075 0 0 -> xyz=0.0 0.045 -0.01725 rpy=-1.57075 0 0
- joint hip_front_rightL_joint: origin xyz=0.0 0.045 -0.030 rpy=-1.57075 0 0 -> xyz=0.0 0.045 -0.01725 rpy=-1.57075 0 0
- joint hip_front_rightR_joint: origin xyz=0.0 0.045 -0.030 rpy=-1.57075 0 0 -> xyz=0.0 0.045 -0.01725 rpy=-1.57075 0 0
- joint motor_back_leftL_joint: origin xyz=-0.20268 0.0455 0 rpy=1.57075 0 3.141592 -> xyz=-0.20268 0.03275 0 rpy=1.57075 0 3.141592
- joint motor_back_leftR_joint: origin xyz=-0.20268 -0.0455 0 rpy=1.57075 0 0 -> xyz=-0.20268 -0.03275 0 rpy=1.57075 0 0
- joint motor_back_rightL_joint: origin xyz=-0.20268 0.0455 0 rpy=1.57075 0 3.141592 -> xyz=-0.20268 0.03275 0 rpy=1.57075 0 3.141592
- joint motor_back_rightR_joint: origin xyz=-0.20268 -0.0455 0 rpy=1.57075 0 0 -> xyz=-0.20268 -0.03275 0 rpy=1.57075 0 0
- joint motor_front_leftL_joint: origin xyz=0.20268 0.0455 0 rpy=1.57075 0 3.141592 -> xyz=0.20268 0.03275 0 rpy=1.57075 0 3.141592
- joint motor_front_leftR_joint: origin xyz=0.20268 -0.0455 0 rpy=1.57075 0 0 -> xyz=0.20268 -0.03275 0 rpy=1.57075 0 0
- joint motor_front_rightL_joint: origin xyz=0.20268 0.0455 0 rpy=1.57075 0 3.141592 -> xyz=0.20268 0.03275 0 rpy=1.57075 0 3.141592
- joint motor_front_rightR_joint: origin xyz=0.20268 -0.0455 0 rpy=1.57075 0 0 -> xyz=0.20268 -0.03275 0 rpy=1.57075 0 0
