Commit message: allow auxilary link to be used for gear btMultiBodyGearConstraint.

File: data/racecar/racecar_differential.urdf (robot description, URDF)
Before this commit: robot racecar, 21 links, 20 joints
Links:
- link chassis: geometry collision mesh filename=meshes/chassis_differential.STL scale=1 1 1 1; visual mesh filename=meshes/chassis_differential.STL scale=1 1 1 1
- link diff2_ring: mass 0.5637 -> 0.0637
- link diff2_sideA: mass 0.556 -> 0.056
- link diff2_sideB: mass 0.556 -> 0.056
- link diff2_spiderA: mass 0.556 -> 0.056
- link diff2_spiderB: mass 0.556 -> 0.056
- link left_front_wheel: mass 0.034055 -> 0.34055
- link left_rear_wheel: mass 0.034055 -> 0.34055
- link right_front_wheel: mass 0.034055 -> 0.34055
- link right_rear_wheel: mass 0.034055 -> 0.34055
