Commit message: improve racecar visuals a little bit with a texture on the wheels

File: data/racecar/racecar.urdf (robot description, URDF)
Before this commit: robot racecar, 13 links, 12 joints
Links:
- link laser: geometry collision box size=0.1 0.1 0.1; visual mesh filename=meshes/hokuyo.obj
- link left_front_wheel: geometry collision cylinder length=0.045 radius=0.05; visual mesh filename=meshes/left_front_wheel.obj
- link left_rear_wheel: geometry collision cylinder length=0.045 radius=0.05; visual mesh filename=meshes/left_rear_wheel.obj
- link right_front_wheel: geometry collision cylinder length=0.045 radius=0.05; visual mesh filename=meshes/right_front_wheel.obj
- link right_rear_wheel: geometry collision cylinder length=0.045 radius=0.05; visual mesh filename=meshes/right_rear_wheel.obj

Commit message: more fixes in pybullet/resources, moved enjoy/train/test in 'examples' folder.

File: data/racecar/racecar.urdf (robot description, URDF)
Before this commit: robot racecar, 13 links, 12 joints
Links:
- link base_link: mass None -> .1
- link chassis: mass None -> .1
