Commit message: update microtaur URDF and example, to be compatible with minitaur_rainbow_dash

File: examples/pybullet/gym/pybullet_data/quadruped/microtaur/microtaur.urdf (robot description, URDF)
Before this commit: robot microtaur, 43 links, 42 joints
Links:
- link lower_leg_back_leftL_link: mass 0.05 -> .086; geometry collision box size=.017 .009 .240; visual box size=.017 .009 .240
- link lower_leg_back_leftR_link: mass 0.05 -> .072; geometry collision box size=.017 .009 .216; visual box size=.017 .009 .216
- link lower_leg_back_rightL_link: mass 0.05 -> .072; geometry collision box size=.017 .009 .216; visual box size=.017 .009 .216
- link lower_leg_back_rightR_link: mass 0.05 -> .086; geometry collision box size=.017 .009 .240; visual box size=.017 .009 .240
- link lower_leg_front_leftL_link: mass 0.05 -> .086; geometry collision box size=.017 .009 .240; visual box size=.017 .009 .240
- link lower_leg_front_leftR_link: mass 0.05 -> .072; geometry collision box size=.017 .009 .216; visual box size=.017 .009 .216
- link lower_leg_front_rightL_link: mass 0.05 -> .072; geometry collision box size=.017 .009 .216; visual box size=.017 .009 .216
- link lower_leg_front_rightR_link: mass 0.05 -> .086; geometry collision box size=.017 .009 .240; visual box size=.017 .009 .240
- link motor_back_leftL_link: mass 0.01 -> .002
- link motor_back_leftR_link: mass 0.01 -> .002
- link motor_back_rightL_link: mass 0.01 -> .002
- link motor_back_rightR_link: mass 0.01 -> .002
- link motor_front_leftL_link: mass 0.01 -> .002
- link motor_front_leftR_link: mass 0.01 -> .002
- link motor_front_rightL_link: mass 0.01 -> .002
- link motor_front_rightR_link: mass 0.01 -> .002; geometry collision cylinder length=0.003 radius=0.0134
- link upper_leg_back_leftL_link: mass 0.05 -> .034; geometry collision box size=.039 .008 .129; visual box size=.039 .008 .129
- link upper_leg_back_leftR_link: mass 0.05 -> .034; geometry collision box size=.039 .008 .129; visual box size=.039 .008 .129
- link upper_leg_back_rightL_link: mass 0.05 -> .034; geometry collision box size=.039 .008 .129; visual box size=.039 .008 .129
- link upper_leg_back_rightR_link: mass 0.05 -> .034; geometry collision box size=.039 .008 .129; visual box size=.039 .008 .129
- link upper_leg_front_leftL_link: mass 0.05 -> .034; geometry collision box size=.039 .008 .129; visual box size=.039 .008 .129
- link upper_leg_front_leftR_link: mass 0.05 -> .034; geometry collision box size=.039 .008 .129; visual box size=.039 .008 .129
- link upper_leg_front_rightL_link: mass 0.05 -> .034; geometry collision box size=.039 .008 .129; visual box size=.039 .008 .129
- link upper_leg_front_rightR_link: mass 0.05 -> .034; geometry collision box size=.039 .008 .129; visual box size=.039 .008 .129
Joints:
- removed joint hip_front_leftR_link
- removed joint hip_front_rightR_link
- removed joint hip_leftR_link
- removed joint hip_rightR_link
- removed joint knee_back_leftL_link
- removed joint knee_back_leftR_link
- removed joint knee_back_rightL_link
- removed joint knee_back_rightR_link
- removed joint knee_front_leftL_link
- removed joint knee_front_leftR_link
- removed joint knee_front_rightL_link
- removed joint knee_front_rightR_link
- removed joint motor_back_leftL_link
- removed joint motor_back_rightL_link
- removed joint motor_front_leftL_link
- removed joint motor_front_rightL_link
- added joint hip_back_leftL_joint: type fixed, parent motor_back_leftL_link, child upper_leg_back_leftL_link, origin xyz=0 .045 -.0145 rpy=-1.57075 0 0, axis 0 0 1, limit effort=100 velocity=100
- added joint hip_back_leftR_joint: type fixed, parent motor_back_leftR_link, child upper_leg_back_leftR_link, origin xyz=0 .045 -.0145 rpy=-1.57075 0 0, axis 0 0 1, limit effort=100 velocity=100
- added joint hip_back_rightL_joint: type fixed, parent motor_back_rightL_link, child upper_leg_back_rightL_link, origin xyz=0 .045 -.0145 rpy=-1.57075 0 0, axis 0 0 1, limit effort=100 velocity=100
- added joint hip_back_rightR_joint: type fixed, parent motor_back_rightR_link, child upper_leg_back_rightR_link, origin xyz=0 .045 -.0145 rpy=-1.57075 0 0, axis 0 0 1, limit effort=100 velocity=100
- added joint hip_front_leftL_joint: type fixed, parent motor_front_leftL_link, child upper_leg_front_leftL_link, origin xyz=0 .045 -.0145 rpy=-1.57075 0 0, axis 0 0 1, limit effort=100 velocity=100
- added joint hip_front_leftR_joint: type fixed, parent motor_front_leftR_link, child upper_leg_front_leftR_link, origin xyz=0 .045 -.0145 rpy=-1.57075 0 0, axis 0 0 1, limit effort=100 velocity=100
- added joint hip_front_rightL_joint: type fixed, parent motor_front_rightL_link, child upper_leg_front_rightL_link, origin xyz=0 .045 -.0145 rpy=-1.57075 0 0, axis 0 0 1, limit effort=100 velocity=100
- added joint hip_front_rightR_joint: type fixed, parent motor_front_rightR_link, child upper_leg_front_rightR_link, origin xyz=0 .045 -.0145 rpy=-1.57075 0 0, axis 0 0 1, limit effort=100 velocity=100
- added joint knee_back_leftL_joint: type continuous, parent upper_leg_back_leftL_link, child lower_leg_back_leftL_link, origin xyz=0 .0085 .056 rpy=0 0 0, axis 0 1 0, limit effort=100 velocity=100
- added joint knee_back_leftR_joint: type continuous, parent upper_leg_back_leftR_link, child lower_leg_back_leftR_link, origin xyz=0 .0085 .056 rpy=0 0 0, axis 0 1 0, limit effort=100 velocity=100
- added joint knee_back_rightL_joint: type continuous, parent upper_leg_back_rightL_link, child lower_leg_back_rightL_link, origin xyz=0 .0085 .056 rpy=0 0 0, axis 0 1 0, limit effort=100 velocity=100
- added joint knee_back_rightR_joint: type continuous, parent upper_leg_back_rightR_link, child lower_leg_back_rightR_link, origin xyz=0 .0085 .056 rpy=0 0 0, axis 0 1 0, limit effort=100 velocity=100
- added joint knee_front_leftL_joint: type continuous, parent upper_leg_front_leftL_link, child lower_leg_front_leftL_link, origin xyz=0 .0085 .056 rpy=0 0 0, axis 0 1 0, limit effort=100 velocity=100
- added joint knee_front_leftR_joint: type continuous, parent upper_leg_front_leftR_link, child lower_leg_front_leftR_link, origin xyz=0 .0085 .056 rpy=0 0 0, axis 0 1 0, limit effort=100 velocity=100
- added joint knee_front_rightL_joint: type continuous, parent upper_leg_front_rightL_link, child lower_leg_front_rightL_link, origin xyz=0 .0085 .056 rpy=0 0 0, axis 0 1 0, limit effort=100 velocity=100
- added joint knee_front_rightR_joint: type continuous, parent upper_leg_front_rightR_link, child lower_leg_front_rightR_link, origin xyz=0 .0085 .056 rpy=0 0 0, axis 0 1 0, limit effort=100 velocity=100
- joint motor_back_leftL_joint: origin xyz=-0.1335 0.035 -0.08 rpy=1.57075 0 3.141592 -> xyz=-0.1335 .0275 -0.08 rpy=1.57075 0 3.141592
- joint motor_back_leftR_joint: origin xyz=-0.1335 -0.03 -0.08 rpy=1.57075 0 0 -> xyz=-0.1335 -.0275 -0.08 rpy=1.57075 0 0
- joint motor_back_rightL_joint: origin xyz=-0.1335 0.03 -0.08 rpy=1.57075 0 3.141592 -> xyz=-0.1335 .0275 -0.08 rpy=1.57075 0 3.141592
- joint motor_back_rightR_joint: origin xyz=-0.1335 -0.035 -0.08 rpy=1.57075 0 0 -> xyz=-0.1335 -.0275 -0.08 rpy=1.57075 0 0
- joint motor_front_leftL_joint: origin xyz=0.1335 0.035 -0.08 rpy=1.57075 0 3.141592 -> xyz=0.1335 .0275 -0.08 rpy=1.57075 0 3.141592
- joint motor_front_leftR_joint: origin xyz=0.1335 -0.03 -0.08 rpy=1.57075 0 0 -> xyz=0.1335 -.0275 -0.08 rpy=1.57075 0 0
- joint motor_front_rightL_joint: origin xyz=0.1335 0.03 -0.08 rpy=1.57075 0 3.141592 -> xyz=0.1335 .0275 -0.08 rpy=1.57075 0 3.141592
- joint motor_front_rightR_joint: origin xyz=0.1335 -0.035 -0.08 rpy=1.57075 0 0 -> xyz=0.1335 -.0275 -0.08 rpy=1.57075 0 0

Commit message: add toe endeffectors for IK of Microtaur

File: examples/pybullet/gym/pybullet_data/quadruped/microtaur/microtaur.urdf (robot description, URDF)
Before this commit: robot microtaur, 43 links, 42 joints
Links:
- added link toe_lower_leg_back_leftL_link, mass 0.01; collision sphere radius=0.01; visual sphere radius=0.01
- added link toe_lower_leg_back_leftR_link, mass 0.01; collision sphere radius=0.01; visual sphere radius=0.01
- added link toe_lower_leg_back_rightL_link, mass 0.01; collision sphere radius=0.01; visual sphere radius=0.01
- added link toe_lower_leg_back_rightR_link, mass 0.01; collision sphere radius=0.01; visual sphere radius=0.01
- added link toe_lower_leg_front_leftL_link, mass 0.01; collision sphere radius=0.01; visual sphere radius=0.01
- added link toe_lower_leg_front_leftR_link, mass 0.01; collision sphere radius=0.01; visual sphere radius=0.01
- added link toe_lower_leg_front_rightL_link, mass 0.01; collision sphere radius=0.01; visual sphere radius=0.01
- added link toe_lower_leg_front_rightR_link, mass 0.01; collision sphere radius=0.01; visual sphere radius=0.01
Joints:
- added joint toe_lower_leg_back_leftL_joint: type fixed, parent lower_leg_back_leftL_link, child toe_lower_leg_back_leftL_link, origin xyz=0 0 0.22
- added joint toe_lower_leg_back_leftR_joint: type fixed, parent lower_leg_back_leftR_link, child toe_lower_leg_back_leftR_link, origin xyz=0 0 0.20
- added joint toe_lower_leg_back_rightL_joint: type fixed, parent lower_leg_back_rightL_link, child toe_lower_leg_back_rightL_link, origin xyz=0 0 0.20
- added joint toe_lower_leg_back_rightR_joint: type fixed, parent lower_leg_back_rightR_link, child toe_lower_leg_back_rightR_link, origin xyz=0 0 0.22
- added joint toe_lower_leg_front_leftL_joint: type fixed, parent lower_leg_front_leftL_link, child toe_lower_leg_front_leftL_link, origin xyz=0 0 0.22
- added joint toe_lower_leg_front_leftR_joint: type fixed, parent lower_leg_front_leftR_link, child toe_lower_leg_front_leftR_link, origin xyz=0 0 0.20
- added joint toe_lower_leg_front_rightL_joint: type fixed, parent lower_leg_front_rightL_link, child toe_lower_leg_front_rightL_link, origin xyz=0 0 0.20
- added joint toe_lower_leg_front_rightR_joint: type fixed, parent lower_leg_front_rightR_link, child toe_lower_leg_front_rightR_link, origin xyz=0 0 0.22
- joint dynamixel4_chassis_front: origin xyz=0 0.135 -0.03 rpy=-1.57079 0 3.141592 -> xyz=0 0.135 -0.03 rpy=-1.57079 0 3.14159265359
- joint dynamixel5_chassis_front: origin xyz=0 -0.055 -0.03 rpy=-1.57079 0 3.141592 -> xyz=0 -0.055 -0.03 rpy=-1.57079 0 3.14159265359
- joint dynamixel7_chassis_rear: origin xyz=0 -0.055 -0.03 rpy=-1.57079 0 3.141592 -> xyz=0 -0.055 -0.03 rpy=-1.57079 0 3.14159265359
- joint dynamixel8_chassis_rear: origin xyz=0 0.135 -0.03 rpy=-1.57079 0 3.141592 -> xyz=0 0.135 -0.03 rpy=-1.57079 0 3.14159265359
- joint hip_back_leftL_joint: origin xyz=0 .045 -.0145 rpy=-1.57075 0 0 -> xyz=0 .045 -.0145 rpy=-1.57079632679 0 0
- joint hip_back_leftR_joint: origin xyz=0 .045 -.0145 rpy=-1.57075 0 0 -> xyz=0 .045 -.0145 rpy=-1.57079632679 0 0
- joint hip_back_rightL_joint: origin xyz=0 .045 -.0145 rpy=-1.57075 0 0 -> xyz=0 .045 -.0145 rpy=-1.57079632679 0 0
- joint hip_back_rightR_joint: origin xyz=0 .045 -.0145 rpy=-1.57075 0 0 -> xyz=0 .045 -.0145 rpy=-1.57079632679 0 0
- joint hip_front_leftL_joint: origin xyz=0 .045 -.0145 rpy=-1.57075 0 0 -> xyz=0 .045 -.0145 rpy=-1.57079632679 0 0
- joint hip_front_leftR_joint: origin xyz=0 .045 -.0145 rpy=-1.57075 0 0 -> xyz=0 .045 -.0145 rpy=-1.57079632679 0 0
- joint hip_front_rightL_joint: origin xyz=0 .045 -.0145 rpy=-1.57075 0 0 -> xyz=0 .045 -.0145 rpy=-1.57079632679 0 0
- joint hip_front_rightR_joint: origin xyz=0 .045 -.0145 rpy=-1.57075 0 0 -> xyz=0 .045 -.0145 rpy=-1.57079632679 0 0
- joint motor_back_leftL_joint: origin xyz=-0.1335 .0275 -0.08 rpy=1.57075 0 3.141592 -> xyz=-0.1335 .0275 -0.08 rpy=1.57079632679 0 3.14159265359
- joint motor_back_leftR_joint: origin xyz=-0.1335 -.0275 -0.08 rpy=1.57075 0 0 -> xyz=-0.1335 -.0275 -0.08 rpy=1.57079632679 0 0
- joint motor_back_rightL_joint: origin xyz=-0.1335 .0275 -0.08 rpy=1.57075 0 3.141592 -> xyz=-0.1335 .0275 -0.08 rpy=1.57079632679 0 3.14159265359
- joint motor_back_rightR_joint: origin xyz=-0.1335 -.0275 -0.08 rpy=1.57075 0 0 -> xyz=-0.1335 -.0275 -0.08 rpy=1.57079632679 0 0
- joint motor_front_leftL_joint: origin xyz=0.1335 .0275 -0.08 rpy=1.57075 0 3.141592 -> xyz=0.1335 .0275 -0.08 rpy=1.57079632679 0 3.14159265359
- joint motor_front_leftR_joint: origin xyz=0.1335 -.0275 -0.08 rpy=1.57075 0 0 -> xyz=0.1335 -.0275 -0.08 rpy=1.57079632679 0 0
- joint motor_front_rightL_joint: origin xyz=0.1335 .0275 -0.08 rpy=1.57075 0 3.141592 -> xyz=0.1335 .0275 -0.08 rpy=1.57079632679 0 3.14159265359
- joint motor_front_rightR_joint: origin xyz=0.1335 -.0275 -0.08 rpy=1.57075 0 0 -> xyz=0.1335 -.0275 -0.08 rpy=1.57079632679 0 0

Commit message: revert to previous leg style of Microtaur

File: examples/pybullet/gym/pybullet_data/quadruped/microtaur/microtaur.urdf (robot description, URDF)
Before this commit: robot microtaur, 51 links, 50 joints
Links:
- link lower_leg_back_leftL_link: mass .086 -> 0.05; geometry collision box size=.01 0.01 .2; visual box size=.01 0.01 .2
- link lower_leg_back_leftR_link: mass .072 -> 0.05; geometry collision box size=.01 0.01 .2032; visual box size=.01 0.01 .2032
- link lower_leg_back_rightL_link: mass .072 -> 0.05; geometry collision box size=.01 0.01 .2; visual box size=.01 0.01 .2
- link lower_leg_back_rightR_link: mass .086 -> 0.05; geometry collision box size=.01 0.01 .2032; visual box size=.01 0.01 .2032
- link lower_leg_front_leftL_link: mass .086 -> 0.05; geometry collision box size=.01 0.01 .198; visual box size=.01 0.01 .198
- link lower_leg_front_leftR_link: mass .072 -> 0.05; geometry collision box size=.01 0.01 .2; visual box size=.01 0.01 .2
- link lower_leg_front_rightL_link: mass .072 -> 0.05; geometry collision box size=.01 0.01 .198; visual box size=.01 0.01 .198
- link lower_leg_front_rightR_link: mass .086 -> 0.05; geometry collision box size=.01 0.01 .2; visual box size=.01 0.01 .2
- link motor_back_leftL_link: mass .002 -> 0.01
- link motor_back_leftR_link: mass .002 -> 0.01
- link motor_back_rightL_link: mass .002 -> 0.01
- link motor_back_rightR_link: mass .002 -> 0.01
- link motor_front_leftL_link: mass .002 -> 0.01
- link motor_front_leftR_link: mass .002 -> 0.01
- link motor_front_rightL_link: mass .002 -> 0.01
- link motor_front_rightR_link: mass .002 -> 0.01; geometry collision cylinder length=0.003 radius=0.0134; visual cylinder length=0.003 radius=0.0134
- link upper_leg_back_leftL_link: mass .034 -> 0.05; geometry collision box size=.01 0.01 .11; visual box size=.01 0.01 .11
- link upper_leg_back_leftR_link: mass .034 -> 0.05; geometry collision box size=.01 0.01 .11; visual box size=.01 0.01 .11
- link upper_leg_back_rightL_link: mass .034 -> 0.05; geometry collision box size=.01 0.01 .11; visual box size=.01 0.01 .11
- link upper_leg_back_rightR_link: mass .034 -> 0.05; geometry collision box size=.01 0.01 .11; visual box size=.01 0.01 .11
- link upper_leg_front_leftL_link: mass .034 -> 0.05; geometry collision box size=.01 0.01 .11; visual box size=.01 0.01 .11
- link upper_leg_front_leftR_link: mass .034 -> 0.05; geometry collision box size=.01 0.01 .11; visual box size=.01 0.01 .11
- link upper_leg_front_rightL_link: mass .034 -> 0.05; geometry collision box size=.01 0.01 .11; visual box size=.01 0.01 .11
- link upper_leg_front_rightR_link: mass .034 -> 0.05; geometry collision box size=.01 0.01 .11; visual box size=.01 0.01 .11
Joints:
- removed joint hip_back_leftR_joint
- removed joint hip_front_rightL_joint
- added joint hip_leftR_joint: type fixed, parent motor_back_leftR_link, child upper_leg_back_leftR_link, origin xyz=0.0 0.06 -0.015 rpy=-1.57075 0 0, axis 0 0 1, limit effort=100 velocity=100
- added joint motor_front_rightL_link: type fixed, parent motor_front_rightL_link, child upper_leg_front_rightL_link, origin xyz=0.0 0.06 -0.015 rpy=-1.57075 0 0, axis 0 0 1, limit effort=100 velocity=100
- joint hip_back_leftL_joint: origin xyz=0 .045 -.0145 rpy=-1.57079632679 0 0 -> xyz=0.0 0.06 -0.015 rpy=-1.57075 0 0
- joint hip_back_rightL_joint: origin xyz=0 .045 -.0145 rpy=-1.57079632679 0 0 -> xyz=0.0 0.06 -0.015 rpy=-1.57075 0 0
- joint hip_back_rightR_joint: origin xyz=0 .045 -.0145 rpy=-1.57079632679 0 0 -> xyz=0.0 0.06 -0.015 rpy=-1.57075 0 0
- joint hip_front_leftL_joint: origin xyz=0 .045 -.0145 rpy=-1.57079632679 0 0 -> xyz=0.0 0.06 -0.015 rpy=-1.57075 0 0
- joint hip_front_leftR_joint: origin xyz=0 .045 -.0145 rpy=-1.57079632679 0 0 -> xyz=0.0 0.06 -0.015 rpy=-1.57075 0 0
- joint hip_front_rightR_joint: origin xyz=0 .045 -.0145 rpy=-1.57079632679 0 0 -> xyz=0.0 0.06 -0.015 rpy=-1.57075 0 0
- joint knee_back_leftL_joint: origin xyz=0 .0085 .056 rpy=0 0 0 -> xyz=0.0 0.01 .055 rpy=0 0 0
- joint knee_back_leftR_joint: origin xyz=0 .0085 .056 rpy=0 0 0 -> xyz=0.0 0.01 .055 rpy=0 0 0
- joint knee_back_rightL_joint: origin xyz=0 .0085 .056 rpy=0 0 0 -> xyz=0.0 0.01 .055 rpy=0 0 0
- joint knee_back_rightR_joint: origin xyz=0 .0085 .056 rpy=0 0 0 -> xyz=0.0 0.01 .055 rpy=0 0 0
- joint knee_front_leftL_joint: origin xyz=0 .0085 .056 rpy=0 0 0 -> xyz=0.0 0.01 .055 rpy=0 0 0
- joint knee_front_leftR_joint: origin xyz=0 .0085 .056 rpy=0 0 0 -> xyz=0.0 0.01 .055 rpy=0 0 0
- joint knee_front_rightL_joint: origin xyz=0 .0085 .056 rpy=0 0 0 -> xyz=0.0 0.01 .055 rpy=0 0 0
- joint knee_front_rightR_joint: origin xyz=0 .0085 .056 rpy=0 0 0 -> xyz=0.0 0.01 .055 rpy=0 0 0
- joint motor_back_leftL_joint: origin xyz=-0.1335 .0275 -0.08 rpy=1.57079632679 0 3.14159265359 -> xyz=-0.1335 0.035 -0.08 rpy=1.57075 0 3.141592
- joint motor_back_leftR_joint: origin xyz=-0.1335 -.0275 -0.08 rpy=1.57079632679 0 0 -> xyz=-0.1335 -0.03 -0.08 rpy=1.57075 0 0
- joint motor_back_rightL_joint: origin xyz=-0.1335 .0275 -0.08 rpy=1.57079632679 0 3.14159265359 -> xyz=-0.1335 0.03 -0.08 rpy=1.57075 0 3.141592
- joint motor_back_rightR_joint: origin xyz=-0.1335 -.0275 -0.08 rpy=1.57079632679 0 0 -> xyz=-0.1335 -0.035 -0.08 rpy=1.57075 0 0
- joint motor_front_leftL_joint: origin xyz=0.1335 .0275 -0.08 rpy=1.57079632679 0 3.14159265359 -> xyz=0.1335 0.035 -0.08 rpy=1.57075 0 3.141592
- joint motor_front_leftR_joint: origin xyz=0.1335 -.0275 -0.08 rpy=1.57079632679 0 0 -> xyz=0.1335 -0.03 -0.08 rpy=1.57075 0 0
- joint motor_front_rightL_joint: origin xyz=0.1335 .0275 -0.08 rpy=1.57079632679 0 3.14159265359 -> xyz=0.1335 0.03 -0.08 rpy=1.57075 0 3.141592
- joint motor_front_rightR_joint: origin xyz=0.1335 -.0275 -0.08 rpy=1.57079632679 0 0 -> xyz=0.1335 -0.035 -0.08 rpy=1.57075 0 0
- joint toe_lower_leg_back_leftL_joint: origin xyz=0 0 0.22 -> xyz=0 0 0.20
- joint toe_lower_leg_back_rightR_joint: origin xyz=0 0 0.22 -> xyz=0 0 0.20
- joint toe_lower_leg_front_leftL_joint: origin xyz=0 0 0.22 -> xyz=0 0 0.20
- joint toe_lower_leg_front_rightR_joint: origin xyz=0 0 0.22 -> xyz=0 0 0.20
