Commit message: also enable simplified convex decomposition collision meshes for xarm6_robot.urdf

File: examples/pybullet/gym/pybullet_data/xarm/xarm6_robot.urdf (robot description, URDF)
Before this commit: robot xarm6, 8 links, 7 joints
Links:
- link link1: geometry collision mesh filename=package://xarm_description/meshes/xarm6/collision/link1_vha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; visual mesh filename=package://xarm_description/meshes/xarm6/visual/link1.stl
- link link2: geometry collision mesh filename=package://xarm_description/meshes/xarm6/collision/link2_vha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; visual mesh filename=package://xarm_description/meshes/xarm6/visual/link2.stl
- link link3: geometry collision mesh filename=package://xarm_description/meshes/xarm6/collision/link3_vha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; visual mesh filename=package://xarm_description/meshes/xarm6/visual/link3.stl
- link link4: geometry collision mesh filename=package://xarm_description/meshes/xarm6/collision/link4_vha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; visual mesh filename=package://xarm_description/meshes/xarm6/visual/link4.stl
- link link5: geometry collision mesh filename=package://xarm_description/meshes/xarm6/collision/link5_vha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; visual mesh filename=package://xarm_description/meshes/xarm6/visual/link5.stl
- link link6: geometry collision mesh filename=package://xarm_description/meshes/xarm6/collision/link6_vha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; visual mesh filename=package://xarm_description/meshes/xarm6/visual/link6.stl
- link link_base: geometry collision mesh filename=package://xarm_description/meshes/xarm6/collision/base_vhac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; visual mesh filename=package://xarm_description/meshes/xarm6/visual/base.stl
