Commit message: remove package from xarm urdfs

File: examples/pybullet/gym/pybullet_data/xarm/base.urdf (robot description, URDF)
Before this commit: robot xarm6_base, 2 links, 1 joints
Links:
- link link_base: geometry collision mesh filename=xarm_description/meshes/xarm6/collision/base_vhacd.obj; visual mesh filename=xarm_description/meshes/xarm6/visual/base.stl

File: examples/pybullet/gym/pybullet_data/xarm/base_com.urdf (robot description, URDF)
Before this commit: robot xarm6_base, 2 links, 1 joints
Links:
- link link_base: geometry collision mesh filename=xarm_description/meshes/xarm6/collision/base_vhacd.obj; visual mesh filename=xarm_description/meshes/xarm6/visual/base.stl

File: examples/pybullet/gym/pybullet_data/xarm/link1.urdf (robot description, URDF)
Before this commit: robot xarm6_link1, 2 links, 1 joints
Links:
- link link1: geometry collision mesh filename=xarm_description/meshes/xarm6/collision/link1_vhacd.obj; visual mesh filename=xarm_description/meshes/xarm6/visual/link1.stl

File: examples/pybullet/gym/pybullet_data/xarm/link1_com.urdf (robot description, URDF)
Before this commit: robot xarm6_link1, 2 links, 1 joints
Links:
- link link1: geometry collision mesh filename=xarm_description/meshes/xarm6/collision/link1_vhacd.obj; visual mesh filename=xarm_description/meshes/xarm6/visual/link1.stl

File: examples/pybullet/gym/pybullet_data/xarm/link2.urdf (robot description, URDF)
Before this commit: robot xarm6_link2, 2 links, 1 joints
Links:
- link link2: geometry collision mesh filename=xarm_description/meshes/xarm6/collision/link2_vhacd.obj; visual mesh filename=xarm_description/meshes/xarm6/visual/link2.stl

File: examples/pybullet/gym/pybullet_data/xarm/link2_com.urdf (robot description, URDF)
Before this commit: robot xarm6_link2, 2 links, 1 joints
Links:
- link link2: geometry collision mesh filename=xarm_description/meshes/xarm6/collision/link2_vhacd.obj; visual mesh filename=xarm_description/meshes/xarm6/visual/link2.stl

File: examples/pybullet/gym/pybullet_data/xarm/link3.urdf (robot description, URDF)
Before this commit: robot xarm6_link3, 2 links, 1 joints
Links:
- link link3: geometry collision mesh filename=xarm_description/meshes/xarm6/collision/link3_vhacd.obj; visual mesh filename=xarm_description/meshes/xarm6/visual/link3.stl

File: examples/pybullet/gym/pybullet_data/xarm/link3_com.urdf (robot description, URDF)
Before this commit: robot xarm6_link3, 2 links, 1 joints
Links:
- link link3: geometry collision mesh filename=xarm_description/meshes/xarm6/collision/link3_vhacd.obj; visual mesh filename=xarm_description/meshes/xarm6/visual/link3.stl

File: examples/pybullet/gym/pybullet_data/xarm/link4.urdf (robot description, URDF)
Before this commit: robot xarm6_link4, 2 links, 1 joints
Links:
- link link4: geometry collision mesh filename=xarm_description/meshes/xarm6/collision/link4_vhacd.obj; visual mesh filename=xarm_description/meshes/xarm6/visual/link4.stl

File: examples/pybullet/gym/pybullet_data/xarm/link4_com.urdf (robot description, URDF)
Before this commit: robot xarm6_link4, 2 links, 1 joints
Links:
- link link4: geometry collision mesh filename=xarm_description/meshes/xarm6/collision/link4_vhacd.obj; visual mesh filename=xarm_description/meshes/xarm6/visual/link4.stl

File: examples/pybullet/gym/pybullet_data/xarm/link5.urdf (robot description, URDF)
Before this commit: robot xarm6_link5, 2 links, 1 joints
Links:
- link link5: geometry collision mesh filename=xarm_description/meshes/xarm6/collision/link5_vhacd.obj; visual mesh filename=xarm_description/meshes/xarm6/visual/link5.stl

File: examples/pybullet/gym/pybullet_data/xarm/link5_com.urdf (robot description, URDF)
Before this commit: robot xarm6_link5, 2 links, 1 joints
Links:
- link link5: geometry collision mesh filename=xarm_description/meshes/xarm6/collision/link5_vhacd.obj; visual mesh filename=xarm_description/meshes/xarm6/visual/link5.stl

File: examples/pybullet/gym/pybullet_data/xarm/link6.urdf (robot description, URDF)
Before this commit: robot xarm6_link6, 2 links, 1 joints
Links:
- link link6: geometry collision mesh filename=xarm_description/meshes/xarm6/collision/link6_vhacd.obj; visual mesh filename=xarm_description/meshes/xarm6/visual/link6.stl

File: examples/pybullet/gym/pybullet_data/xarm/link6_com.urdf (robot description, URDF)
Before this commit: robot xarm6_link6, 2 links, 1 joints
Links:
- link link6: geometry collision mesh filename=xarm_description/meshes/xarm6/collision/link6_vhacd.obj; visual mesh filename=xarm_description/meshes/xarm6/visual/link6.stl

File: examples/pybullet/gym/pybullet_data/xarm/xarm6_robot.urdf (robot description, URDF)
Before this commit: robot xarm6, 8 links, 7 joints
Links:
- link link1: geometry collision mesh filename=xarm_description/meshes/xarm6/collision/link1_vhacd.obj; visual mesh filename=xarm_description/meshes/xarm6/visual/link1.stl
- link link2: geometry collision mesh filename=xarm_description/meshes/xarm6/collision/link2_vhacd.obj; visual mesh filename=xarm_description/meshes/xarm6/visual/link2.stl
- link link3: geometry collision mesh filename=xarm_description/meshes/xarm6/collision/link3_vhacd.obj; visual mesh filename=xarm_description/meshes/xarm6/visual/link3.stl
- link link4: geometry collision mesh filename=xarm_description/meshes/xarm6/collision/link4_vhacd.obj; visual mesh filename=xarm_description/meshes/xarm6/visual/link4.stl
- link link5: geometry collision mesh filename=xarm_description/meshes/xarm6/collision/link5_vhacd.obj; visual mesh filename=xarm_description/meshes/xarm6/visual/link5.stl
- link link6: geometry collision mesh filename=xarm_description/meshes/xarm6/collision/link6_vhacd.obj; visual mesh filename=xarm_description/meshes/xarm6/visual/link6.stl
- link link_base: geometry collision mesh filename=xarm_description/meshes/xarm6/collision/base_vhacd.obj; visual mesh filename=xarm_description/meshes/xarm6/visual/base.stl

File: examples/pybullet/gym/pybullet_data/xarm/xarm6_robot_white.urdf (robot description, URDF)
Before this commit: robot xarm6, 8 links, 7 joints
Links:
- link link1: geometry collision mesh filename=xarm_description/meshes/xarm6/collision/link1_vhacd.obj; visual mesh filename=xarm_description/meshes/xarm6/visual/link1.stl
- link link2: geometry collision mesh filename=xarm_description/meshes/xarm6/collision/link2_vhacd.obj; visual mesh filename=xarm_description/meshes/xarm6/visual/link2.stl
- link link3: geometry collision mesh filename=xarm_description/meshes/xarm6/collision/link3_vhacd.obj; visual mesh filename=xarm_description/meshes/xarm6/visual/link3.stl
- link link4: geometry collision mesh filename=xarm_description/meshes/xarm6/collision/link4_vhacd.obj; visual mesh filename=xarm_description/meshes/xarm6/visual/link4.stl
- link link5: geometry collision mesh filename=xarm_description/meshes/xarm6/collision/link5_vhacd.obj; visual mesh filename=xarm_description/meshes/xarm6/visual/link5.stl
- link link6: geometry collision mesh filename=xarm_description/meshes/xarm6/collision/link6_vhacd.obj; visual mesh filename=xarm_description/meshes/xarm6/visual/link6.stl
- link link_base: geometry collision mesh filename=xarm_description/meshes/xarm6/collision/base_vhacd.obj; visual mesh filename=xarm_description/meshes/xarm6/visual/base.stl

File: examples/pybullet/gym/pybullet_data/xarm/xarm6_with_gripper.urdf (robot description, URDF)
Before this commit: robot xarm6_with_gripper, 15 links, 14 joints
Links:
- link link1: geometry collision mesh filename=xarm_description/meshes/xarm6/collision/link1_vhacd.obj; visual mesh filename=xarm_description/meshes/xarm6/visual/link1.stl
- link link2: geometry collision mesh filename=xarm_description/meshes/xarm6/collision/link2_vhacd2.obj; visual mesh filename=xarm_description/meshes/xarm6/visual/link2.stl
- link link3: geometry collision mesh filename=xarm_description/meshes/xarm6/collision/link3_vhacd.obj; visual mesh filename=xarm_description/meshes/xarm6/visual/link3.stl
- link link4: geometry collision mesh filename=xarm_description/meshes/xarm6/collision/link4_vhacd.obj; visual mesh filename=xarm_description/meshes/xarm6/visual/link4.stl
- link link5: geometry collision mesh filename=xarm_description/meshes/xarm6/collision/link5_vhacd.obj; visual mesh filename=xarm_description/meshes/xarm6/visual/link5.stl
- link link6: geometry collision mesh filename=xarm_description/meshes/xarm6/visual/link6.stl; visual mesh filename=xarm_description/meshes/xarm6/visual/link6.stl
- link link_base: geometry collision mesh filename=xarm_description/meshes/xarm6/collision/base_vhacd.obj; visual mesh filename=xarm_description/meshes/xarm6/visual/base.stl
