Commit message: remove package xarm_gripper from xarm urdfs

File: examples/pybullet/gym/pybullet_data/xarm/xarm6_with_gripper.urdf (robot description, URDF)
Before this commit: robot xarm6_with_gripper, 15 links, 14 joints
Links:
- link left_finger: geometry collision mesh filename=xarm_gripper/meshes/left_finger.STL; visual mesh filename=xarm_gripper/meshes/left_finger.STL
- link left_inner_knuckle: geometry collision mesh filename=xarm_gripper/meshes/left_inner_knuckle.STL; visual mesh filename=xarm_gripper/meshes/left_inner_knuckle.STL
- link left_outer_knuckle: geometry collision mesh filename=xarm_gripper/meshes/left_outer_knuckle.STL; visual mesh filename=xarm_gripper/meshes/left_outer_knuckle.STL
- link right_finger: geometry collision mesh filename=xarm_gripper/meshes/right_finger.STL; visual mesh filename=xarm_gripper/meshes/right_finger.STL
- link right_inner_knuckle: geometry collision mesh filename=xarm_gripper/meshes/right_inner_knuckle.STL; visual mesh filename=xarm_gripper/meshes/right_inner_knuckle.STL
- link right_outer_knuckle: geometry collision mesh filename=xarm_gripper/meshes/right_outer_knuckle.STL; visual mesh filename=xarm_gripper/meshes/right_outer_knuckle.STL
- link xarm_gripper_base_link: geometry collision mesh filename=xarm_gripper/meshes/base_link.STL; visual mesh filename=xarm_gripper/meshes/base_link.STL
