Commit message: update a1 urdf to match naming for our software update test a1.py script

File: examples/pybullet/gym/pybullet_data/a1/a1.urdf (robot description, URDF)
Before this commit: robot a1_description, 23 links, 22 joints
Links:
- removed link FL_calf
- removed link FL_foot
- removed link FL_thigh
- removed link FL_thigh_shoulder
- removed link FR_calf
- removed link FR_foot
- removed link FR_thigh
- removed link FR_thigh_shoulder
- removed link RL_calf
- removed link RL_foot
- removed link RL_thigh
- removed link RL_thigh_shoulder
- removed link RR_calf
- removed link RR_foot
- removed link RR_thigh
- removed link RR_thigh_shoulder
- removed link base
- added link FL_lower, mass 0.166; collision box size=0.2 0.016 0.016; visual mesh filename=meshes/calf.obj scale=1 1 1
- added link FL_toe, mass 0.06; collision sphere radius=0.02; visual sphere radius=0.01
- added link FL_upper, mass 1.013; collision box size=0.2 0.0245 0.034; visual mesh filename=meshes/thigh.obj scale=1 1 1
- added link FL_upper_shoulder; collision cylinder length=0.032 radius=0.041
- added link FR_lower, mass 0.166; collision box size=0.2 0.016 0.016; visual mesh filename=meshes/calf.obj scale=1 1 1
- added link FR_toe, mass 0.06; collision sphere radius=0.02; visual sphere radius=0.01
- added link FR_upper, mass 1.013; collision box size=0.2 0.0245 0.034; visual mesh filename=meshes/thigh_mirror.obj scale=1 1 1
- added link FR_upper_shoulder; collision cylinder length=0.032 radius=0.041
- added link RL_lower, mass 0.166; collision box size=0.2 0.016 0.016; visual mesh filename=meshes/calf.obj scale=1 1 1
- added link RL_toe, mass 0.06; collision sphere radius=0.02; visual sphere radius=0.01
- added link RL_upper, mass 1.013; collision box size=0.2 0.0245 0.034; visual mesh filename=meshes/thigh.obj scale=1 1 1
- added link RL_upper_shoulder; collision cylinder length=0.032 radius=0.041
- added link RR_lower, mass 0.166; collision box size=0.2 0.016 0.016; visual mesh filename=meshes/calf.obj scale=1 1 1
- added link RR_toe, mass 0.06; collision sphere radius=0.02; visual sphere radius=0.01
- added link RR_upper, mass 1.013; collision box size=0.2 0.0245 0.034; visual mesh filename=meshes/thigh_mirror.obj scale=1 1 1
- added link RR_upper_shoulder; collision cylinder length=0.032 radius=0.041
Joints:
- removed joint FL_calf_joint
- removed joint FL_foot_fixed
- removed joint FL_thigh_joint
- removed joint FR_calf_joint
- removed joint FR_foot_fixed
- removed joint FR_thigh_joint
- removed joint RL_calf_joint
- removed joint RL_foot_fixed
- removed joint RL_thigh_joint
- removed joint RR_calf_joint
- removed joint RR_foot_fixed
- removed joint RR_thigh_joint
- removed joint floating_base
- added joint FL_lower_joint: type revolute, parent FL_upper, child FL_lower, origin xyz=0 0 -0.2 rpy=0 0 0, axis 0 1 0, limit lower=-2.69653369433 upper=-0.916297857297 effort=55 velocity=28.6
- added joint FL_toe_fixed: type fixed, parent FL_lower, child FL_toe, origin xyz=0 0 -0.2 rpy=0 0 0
- added joint FL_upper_joint: type revolute, parent FL_hip, child FL_upper, origin xyz=0 0.08505 0 rpy=0 0 0, axis 0 1 0, limit lower=-1.0471975512 upper=4.18879020479 effort=55 velocity=28.6
- added joint FR_lower_joint: type revolute, parent FR_upper, child FR_lower, origin xyz=0 0 -0.2 rpy=0 0 0, axis 0 1 0, limit lower=-2.69653369433 upper=-0.916297857297 effort=55 velocity=28.6
- added joint FR_toe_fixed: type fixed, parent FR_lower, child FR_toe, origin xyz=0 0 -0.2 rpy=0 0 0
- added joint FR_upper_joint: type revolute, parent FR_hip, child FR_upper, origin xyz=0 -0.08505 0 rpy=0 0 0, axis 0 1 0, limit lower=-1.0471975512 upper=4.18879020479 effort=55 velocity=28.6
- added joint RL_lower_joint: type revolute, parent RL_upper, child RL_lower, origin xyz=0 0 -0.2 rpy=0 0 0, axis 0 1 0, limit lower=-2.69653369433 upper=-0.916297857297 effort=55 velocity=28.6
- added joint RL_toe_fixed: type fixed, parent RL_lower, child RL_toe, origin xyz=0 0 -0.2 rpy=0 0 0
- added joint RL_upper_joint: type revolute, parent RL_hip, child RL_upper, origin xyz=0 0.08505 0 rpy=0 0 0, axis 0 1 0, limit lower=-1.0471975512 upper=4.18879020479 effort=55 velocity=28.6
- added joint RR_lower_joint: type revolute, parent RR_upper, child RR_lower, origin xyz=0 0 -0.2 rpy=0 0 0, axis 0 1 0, limit lower=-2.69653369433 upper=-0.916297857297 effort=55 velocity=28.6
- added joint RR_toe_fixed: type fixed, parent RR_lower, child RR_toe, origin xyz=0 0 -0.2 rpy=0 0 0
- added joint RR_upper_joint: type revolute, parent RR_hip, child RR_upper, origin xyz=0 -0.08505 0 rpy=0 0 0, axis 0 1 0, limit lower=-1.0471975512 upper=4.18879020479 effort=55 velocity=28.6
- joint FL_hip_fixed: child FL_thigh_shoulder -> FL_upper_shoulder
- joint FR_hip_fixed: child FR_thigh_shoulder -> FR_upper_shoulder
- joint RL_hip_fixed: child RL_thigh_shoulder -> RL_upper_shoulder
- joint RR_hip_fixed: child RR_thigh_shoulder -> RR_upper_shoulder
