Commit message: Change Aliengo urdf naming & add example script

File: examples/pybullet/gym/pybullet_data/aliengo/aliengo.urdf (robot description, URDF)
Before this commit: robot aliengo_description, 19 links, 18 joints
Links:
- removed link FL_calf
- removed link FL_foot
- removed link FL_thigh
- removed link FR_calf
- removed link FR_foot
- removed link FR_thigh
- removed link RL_calf
- removed link RL_foot
- removed link RL_thigh
- removed link RR_calf
- removed link RR_foot
- removed link RR_thigh
- removed link base
- added link FL_lower, mass 0.207; collision box size=0.25 0.0208 0.016; visual mesh filename=meshes/calf.stl scale=1 1 1
- added link FL_toe, mass 0.06; collision sphere radius=0.0265; visual sphere radius=0.0165
- added link FL_upper, mass 0.639; collision box size=0.25 0.0374 0.043; visual mesh filename=meshes/thigh.stl scale=1 1 1
- added link FR_lower, mass 0.207; collision box size=0.25 0.0208 0.016; visual mesh filename=meshes/calf.stl scale=1 1 1
- added link FR_toe, mass 0.06; collision sphere radius=0.0265; visual sphere radius=0.0165
- added link FR_upper, mass 0.639; collision box size=0.25 0.0374 0.043; visual mesh filename=meshes/thigh_mirror.stl scale=1 1 1
- added link RL_lower, mass 0.207; collision box size=0.25 0.0208 0.016; visual mesh filename=meshes/calf.stl scale=1 1 1
- added link RL_toe, mass 0.06; collision sphere radius=0.0265; visual sphere radius=0.0165
- added link RL_upper, mass 0.639; collision box size=0.25 0.0374 0.043; visual mesh filename=meshes/thigh.stl scale=1 1 1
- added link RR_lower, mass 0.207; collision box size=0.25 0.0208 0.016; visual mesh filename=meshes/calf.stl scale=1 1 1
- added link RR_toe, mass 0.06; collision sphere radius=0.0265; visual sphere radius=0.0165
- added link RR_upper, mass 0.639; collision box size=0.25 0.0374 0.043; visual mesh filename=meshes/thigh_mirror.stl scale=1 1 1
Joints:
- removed joint FL_calf_joint
- removed joint FL_foot_fixed
- removed joint FL_thigh_joint
- removed joint FR_calf_joint
- removed joint FR_foot_fixed
- removed joint FR_thigh_joint
- removed joint RL_calf_joint
- removed joint RL_foot_fixed
- removed joint RL_thigh_joint
- removed joint RR_calf_joint
- removed joint RR_foot_fixed
- removed joint RR_thigh_joint
- removed joint floating_base
- added joint FL_lower_joint: type revolute, parent FL_upper, child FL_lower, origin xyz=0 0 -0.25 rpy=0 0 0, axis 0 1 0, limit lower=-2.77507351067 upper=-0.645771823238 effort=44.4 velocity=40
- added joint FL_toe_fixed: type fixed, parent FL_lower, child FL_toe, origin xyz=0 0 -0.25 rpy=0 0 0
- added joint FL_upper_joint: type continuous, parent FL_hip, child FL_upper, origin xyz=0 0.083 0 rpy=0 0 0, axis 0 1 0, limit effort=44.4 velocity=40
- added joint FR_lower_joint: type revolute, parent FR_upper, child FR_lower, origin xyz=0 0 -0.25 rpy=0 0 0, axis 0 1 0, limit lower=-2.77507351067 upper=-0.645771823238 effort=44.4 velocity=40
- added joint FR_toe_fixed: type fixed, parent FR_lower, child FR_toe, origin xyz=0 0 -0.25 rpy=0 0 0
- added joint FR_upper_joint: type continuous, parent FR_hip, child FR_upper, origin xyz=0 -0.083 0 rpy=0 0 0, axis 0 1 0, limit effort=44.4 velocity=40
- added joint RL_lower_joint: type revolute, parent RL_upper, child RL_lower, origin xyz=0 0 -0.25 rpy=0 0 0, axis 0 1 0, limit lower=-2.77507351067 upper=-0.645771823238 effort=44.4 velocity=40
- added joint RL_toe_fixed: type fixed, parent RL_lower, child RL_toe, origin xyz=0 0 -0.25 rpy=0 0 0
- added joint RL_upper_joint: type continuous, parent RL_hip, child RL_upper, origin xyz=0 0.083 0 rpy=0 0 0, axis 0 1 0, limit effort=44.4 velocity=40
- added joint RR_lower_joint: type revolute, parent RR_upper, child RR_lower, origin xyz=0 0 -0.25 rpy=0 0 0, axis 0 1 0, limit lower=-2.77507351067 upper=-0.645771823238 effort=44.4 velocity=40
- added joint RR_toe_fixed: type fixed, parent RR_lower, child RR_toe, origin xyz=0 0 -0.25 rpy=0 0 0
- added joint RR_upper_joint: type continuous, parent RR_hip, child RR_upper, origin xyz=0 -0.083 0 rpy=0 0 0, axis 0 1 0, limit effort=44.4 velocity=40

Commit message: delete MPL licensed meshes, replace by manual textured meshes.

File: examples/pybullet/gym/pybullet_data/aliengo/aliengo.urdf (robot description, URDF)
Before this commit: robot aliengo_description, 18 links, 17 joints
Links:
- link FL_hip: geometry collision cylinder length=0.0418 radius=0.046; visual mesh filename=meshes/hip.obj scale=1 1 1
- link FL_lower: geometry collision box size=0.25 0.0208 0.016; visual mesh filename=meshes/calf.obj scale=1 1 1
- link FL_upper: geometry collision box size=0.25 0.0374 0.043; visual mesh filename=meshes/thigh.obj scale=1 1 1
- link FR_hip: geometry collision cylinder length=0.0418 radius=0.046; visual mesh filename=meshes/hip.obj scale=1 1 1
- link FR_lower: geometry collision box size=0.25 0.0208 0.016; visual mesh filename=meshes/calf.obj scale=1 1 1
- link FR_upper: geometry collision box size=0.25 0.0374 0.043; visual mesh filename=meshes/thigh_mirror.obj scale=1 1 1
- link RL_hip: geometry collision cylinder length=0.0418 radius=0.046; visual mesh filename=meshes/hip.obj scale=1 1 1
- link RL_lower: geometry collision box size=0.25 0.0208 0.016; visual mesh filename=meshes/calf.obj scale=1 1 1
- link RL_upper: geometry collision box size=0.25 0.0374 0.043; visual mesh filename=meshes/thigh.obj scale=1 1 1
- link RR_hip: geometry collision cylinder length=0.0418 radius=0.046; visual mesh filename=meshes/hip.obj scale=1 1 1
- link RR_lower: geometry collision box size=0.25 0.0208 0.016; visual mesh filename=meshes/calf.obj scale=1 1 1
- link RR_upper: geometry collision box size=0.25 0.0374 0.043; visual mesh filename=meshes/thigh_mirror.obj scale=1 1 1
- link trunk: geometry collision box size=0.647 0.15 0.112; visual mesh filename=meshes/trunk.obj scale=1 1 1
