Commit message: Fix differential references in racecar

File: examples/pybullet/gym/pybullet_data/racecar/racecar_differential.urdf (robot description, URDF)
Before this commit: robot racecar, 21 links, 20 joints
Links:
- link diff2_ring: geometry collision cylinder length=0.01 radius=0.025; visual mesh filename=../differential/diff_carrier.stl scale=0.001 0.001 0.001
- link diff2_sideA: geometry collision cylinder length=0.01 radius=0.015; visual mesh filename=../differential/diff_side.stl scale=0.001 0.001 0.001
- link diff2_sideB: geometry collision cylinder length=0.01 radius=0.015; visual mesh filename=../differential/diff_side.stl scale=0.001 0.001 0.001
- link diff2_spiderA: geometry collision cylinder length=0.01 radius=0.015; visual mesh filename=../differential/diff_spider.stl scale=0.001 0.001 0.001
- link diff2_spiderB: geometry collision cylinder length=0.01 radius=0.015; visual mesh filename=../differential/diff_spider.stl scale=0.001 0.001 0.001
- link diff_ring: geometry collision cylinder length=0.01 radius=0.025; visual mesh filename=../differential/diff_carrier.stl scale=0.001 0.001 0.001
- link diff_sideA: geometry collision cylinder length=0.01 radius=0.015; visual mesh filename=../differential/diff_side.stl scale=0.001 0.001 0.001
- link diff_sideB: geometry collision cylinder length=0.01 radius=0.015; visual mesh filename=../differential/diff_side.stl scale=0.001 0.001 0.001
- link diff_spiderA: geometry collision cylinder length=0.01 radius=0.015; visual mesh filename=../differential/diff_spider.stl scale=0.001 0.001 0.001
- link diff_spiderB: geometry collision cylinder length=0.01 radius=0.015; visual mesh filename=../differential/diff_spider.stl scale=0.001 0.001 0.001
