Commit message: Fix differential reference

File: examples/pybullet/gym/pybullet_data/differential/diff_ring.urdf (robot description, URDF)
Before this commit: robot husky_robot, 6 links, 5 joints
Links:
- link diff_ring: geometry collision cylinder length=0.01 radius=0.05; visual mesh filename=diff_carrier.stl scale=0.001 0.001 0.001
- link diff_sideA: geometry collision cylinder length=0.01 radius=0.015; visual mesh filename=diff_side.stl scale=0.001 0.001 0.001
- link diff_sideB: geometry collision cylinder length=0.01 radius=0.015; visual mesh filename=diff_side.stl scale=0.001 0.001 0.001
- link diff_spiderA: geometry collision cylinder length=0.01 radius=0.015; visual mesh filename=diff_spider.stl scale=0.001 0.001 0.001
- link diff_spiderB: geometry collision cylinder length=0.01 radius=0.015; visual mesh filename=diff_spider.stl scale=0.001 0.001 0.001
